File: EIM/pcb/EIM/RS485.kicad_sch (KiCad schematic)
At the start: 9 parts, among them IC2 SN65HVD1780QDRQ1

Commit message: added Arjun's comments, assigned some MCU pins
Parts:
- renumbered C30 to C36, D2 to D12, R13 to R18, R14 to R19, R12 to R20, R10 to R21, R11 to R22
Changed lines of the file:
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@@
 		(on_board yes)
 		(dnp no)
-		(property "Reference" "#PWR051"
+		(property "Reference" "#PWR088"
 			(at 166.37 74.93 0)
 			(effects
@@
 			(project "EIM"
 				(path "/2e0b3b3d-5537-41dc-9fad-4fb33afdbfad/458a1c59-d9de-4aa8-ac53-f47317918c09"
-					(reference "#PWR051")
+					(reference "#PWR088")
 					(unit 1)
 				)
@@
 		(on_board yes)
 		(dnp no)
-		(property "Reference" "R14"
+		(property "Reference" "R19"
 			(at 125.984 67.056 0)
 			(effects
@@
 			(project "EIM"
 				(path "/2e0b3b3d-5537-41dc-9fad-4fb33afdbfad/458a1c59-d9de-4aa8-ac53-f47317918c09"
-					(reference "R14")
+					(reference "R19")
 					(unit 1)
 				)
@@
 		(on_board yes)
 		(dnp no)
-		(property "Reference" "R10"
+		(property "Reference" "R21"
 			(at 184.404 84.328 90)
 			(effects
@@
 			(project "EIM"
 				(path "/2e0b3b3d-5537-41dc-9fad-4fb33afdbfad/458a1c59-d9de-4aa8-ac53-f47317918c09"
-					(reference "R10")
+					(reference "R21")
 					(unit 1)
 				)
@@
 		(on_board yes)
 		(dnp no)
-		(property "Reference" "#PWR052"
+		(property "Reference" "#PWR089"
 			(at 166.37 88.9 0)
 			(effects
@@
 			(project "EIM"
 				(path "/2e0b3b3d-5537-41dc-9fad-4fb33afdbfad/458a1c59-d9de-4aa8-ac53-f47317918c09"
-					(reference "#PWR052")
+					(reference "#PWR089")
 					(unit 1)
 				)
@@
 		(on_board yes)
 		(dnp no)
-		(property "Reference" "C30"
+		(property "Reference" "C36"
 			(at 166.878 81.534 0)
 			(effects
@@
 			(project "EIM"
 				(path "/2e0b3b3d-5537-41dc-9fad-4fb33afdbfad/458a1c59-d9de-4aa8-ac53-f47317918c09"
-					(reference "C30")
+					(reference "C36")
 					(unit 1)
 				)
@@
 		(on_board yes)
 		(dnp no)
-		(property "Reference" "R11"
+		(property "Reference" "R22"
 			(at 184.404 102.108 90)
 			(effects
@@
 			(project "EIM"
 				(path "/2e0b3b3d-5537-41dc-9fad-4fb33afdbfad/458a1c59-d9de-4aa8-ac53-f47317918c09"
-					(reference "R11")
+					(reference "R22")
 					(unit 1)
 				)
@@
 		(on_board yes)
 		(dnp no)
-		(property "Reference" "#PWR054"
+		(property "Reference" "#PWR087"
 			(at 123.19 64.77 0)
 			(effects
@@
 			(project "EIM"
 				(path "/2e0b3b3d-5537-41dc-9fad-4fb33afdbfad/458a1c59-d9de-4aa8-ac53-f47317918c09"
-					(reference "#PWR054")
+					(reference "#PWR087")
 					(unit 1)
 				)
@@
 		(on_board yes)
 		(dnp no)
-		(property "Reference" "#PWR053"
+		(property "Reference" "#PWR090"
 			(at 166.37 111.76 0)
 			(effects
@@
 			(project "EIM"
 				(path "/2e0b3b3d-5537-41dc-9fad-4fb33afdbfad/458a1c59-d9de-4aa8-ac53-f47317918c09"
-					(reference "#PWR053")
+					(reference "#PWR090")
 					(unit 1)
 				)
@@
 		(dnp no)
 		(fields_autoplaced yes)
-		(property "Reference" "D2"
+		(property "Reference" "D12"
 			(at 196.85 93.9799 90)
 			(effects
@@
 			(project ""
 				(path "/2e0b3b3d-5537-41dc-9fad-4fb33afdbfad/458a1c59-d9de-4aa8-ac53-f47317918c09"
-					(reference "D2")
+					(reference "D12")
 					(unit 1)
 				)
@@
 		(on_board yes)
 		(dnp no)
-		(property "Reference" "R13"
+		(property "Reference" "R18"
 			(at 114.808 97.536 90)
 			(effects
@@
 			(project "EIM"
 				(path "/2e0b3b3d-5537-41dc-9fad-4fb33afdbfad/458a1c59-d9de-4aa8-ac53-f47317918c09"
-					(reference "R13")
+					(reference "R18")
 					(unit 1)
 				)
@@
 		(on_board yes)
 		(dnp no)
-		(property "Reference" "R12"
+		(property "Reference" "R20"
 			(at 160.02 126.238 90)
 			(effects
@@
 			(project "EIM"
 				(path "/2e0b3b3d-5537-41dc-9fad-4fb33afdbfad/458a1c59-d9de-4aa8-ac53-f47317918c09"
-					(reference "R12")
+					(reference "R20")
 					(unit 1)
 				)
@@
 		(on_board yes)
 		(dnp no)
-		(property "Reference" "#PWR055"
+		(property "Reference" "#PWR086"
 			(at 116.84 107.95 0)
 			(effects
@@
 			(project "EIM"
 				(path "/2e0b3b3d-5537-41dc-9fad-4fb33afdbfad/458a1c59-d9de-4aa8-ac53-f47317918c09"
-					(reference "#PWR055")
+					(reference "#PWR086")
 					(unit 1)
 				)
@@
 		(on_board yes)
 		(dnp no)
-		(property "Reference" "#PWR050"
+		(property "Reference" "#PWR091"
 			(at 184.15 95.25 0)
 			(effects
@@
 			(project ""
 				(path "/2e0b3b3d-5537-41dc-9fad-4fb33afdbfad/458a1c59-d9de-4aa8-ac53-f47317918c09"
-					(reference "#PWR050")
-					(unit 1)
-				)
+					(reference "#PWR091")
+					(unit 1)
+				)

Commit message: Layout 75% done, before 8V bus deletion
Parts:
- renumbered C36 to C43, D12 to D14, JP3 to JP4, R18 to R22, R19 to R23, R20 to R24, R21 to R25, R22 to R26
Changed lines of the file:
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@@
 		(on_board yes)
 		(dnp no)
-		(property "Reference" "#PWR088"
+		(property "Reference" "#PWR097"
 			(at 166.37 74.93 0)
 			(effects
@@
 			(project "EIM"
 				(path "/2e0b3b3d-5537-41dc-9fad-4fb33afdbfad/458a1c59-d9de-4aa8-ac53-f47317918c09"
-					(reference "#PWR088")
+					(reference "#PWR097")
 					(unit 1)
 				)
@@
 		(dnp no)
 		(fields_autoplaced yes)
-		(property "Reference" "JP3"
+		(property "Reference" "JP4"
 			(at 151.13 121.92 0)
 			(effects
@@
 			(project "EIM"
 				(path "/2e0b3b3d-5537-41dc-9fad-4fb33afdbfad/458a1c59-d9de-4aa8-ac53-f47317918c09"
-					(reference "JP3")
+					(reference "JP4")
 					(unit 1)
 				)
@@
 		(on_board yes)
 		(dnp no)
-		(property "Reference" "R19"
+		(property "Reference" "R23"
 			(at 125.984 67.056 0)
 			(effects
@@
 			(project "EIM"
 				(path "/2e0b3b3d-5537-41dc-9fad-4fb33afdbfad/458a1c59-d9de-4aa8-ac53-f47317918c09"
-					(reference "R19")
+					(reference "R23")
 					(unit 1)
 				)
@@
 		(on_board yes)
 		(dnp no)
-		(property "Reference" "R21"
+		(property "Reference" "R25"
 			(at 184.404 84.328 90)
 			(effects
@@
 			(project "EIM"
 				(path "/2e0b3b3d-5537-41dc-9fad-4fb33afdbfad/458a1c59-d9de-4aa8-ac53-f47317918c09"
-					(reference "R21")
+					(reference "R25")
 					(unit 1)
 				)
@@
 		(on_board yes)
 		(dnp no)
-		(property "Reference" "#PWR089"
+		(property "Reference" "#PWR098"
 			(at 166.37 88.9 0)
 			(effects
@@
 			(project "EIM"
 				(path "/2e0b3b3d-5537-41dc-9fad-4fb33afdbfad/458a1c59-d9de-4aa8-ac53-f47317918c09"
-					(reference "#PWR089")
+					(reference "#PWR098")
 					(unit 1)
 				)
@@
 		(on_board yes)
 		(dnp no)
-		(property "Reference" "C36"
+		(property "Reference" "C43"
 			(at 166.878 81.534 0)
 			(effects
@@
 			(project "EIM"
 				(path "/2e0b3b3d-5537-41dc-9fad-4fb33afdbfad/458a1c59-d9de-4aa8-ac53-f47317918c09"
-					(reference "C36")
+					(reference "C43")
 					(unit 1)
 				)
@@
 		(on_board yes)
 		(dnp no)
-		(property "Reference" "R22"
+		(property "Reference" "R26"
 			(at 184.404 102.108 90)
 			(effects
@@
 			(project "EIM"
 				(path "/2e0b3b3d-5537-41dc-9fad-4fb33afdbfad/458a1c59-d9de-4aa8-ac53-f47317918c09"
-					(reference "R22")
+					(reference "R26")
 					(unit 1)
 				)
@@
 		(on_board yes)
 		(dnp no)
-		(property "Reference" "#PWR087"
+		(property "Reference" "#PWR096"
 			(at 123.19 64.77 0)
 			(effects
@@
 			(project "EIM"
 				(path "/2e0b3b3d-5537-41dc-9fad-4fb33afdbfad/458a1c59-d9de-4aa8-ac53-f47317918c09"
-					(reference "#PWR087")
+					(reference "#PWR096")
 					(unit 1)
 				)
@@
 		(on_board yes)
 		(dnp no)
-		(property "Reference" "#PWR090"
+		(property "Reference" "#PWR099"
 			(at 166.37 111.76 0)
 			(effects
@@
 			(project "EIM"
 				(path "/2e0b3b3d-5537-41dc-9fad-4fb33afdbfad/458a1c59-d9de-4aa8-ac53-f47317918c09"
-					(reference "#PWR090")
+					(reference "#PWR099")
 					(unit 1)
 				)
@@
 		(dnp no)
 		(fields_autoplaced yes)
-		(property "Reference" "D12"
+		(property "Reference" "D14"
 			(at 196.85 93.9799 90)
 			(effects
@@
 			(project ""
 				(path "/2e0b3b3d-5537-41dc-9fad-4fb33afdbfad/458a1c59-d9de-4aa8-ac53-f47317918c09"
-					(reference "D12")
+					(reference "D14")
 					(unit 1)
 				)
@@
 		(on_board yes)
 		(dnp no)
-		(property "Reference" "R18"
+		(property "Reference" "R22"
 			(at 114.808 97.536 90)
 			(effects
@@
 			(project "EIM"
 				(path "/2e0b3b3d-5537-41dc-9fad-4fb33afdbfad/458a1c59-d9de-4aa8-ac53-f47317918c09"
-					(reference "R18")
+					(reference "R22")
 					(unit 1)
 				)
@@
 		(on_board yes)
 		(dnp no)
-		(property "Reference" "R20"
+		(property "Reference" "R24"
 			(at 160.02 126.238 90)
 			(effects
@@
 			(project "EIM"
 				(path "/2e0b3b3d-5537-41dc-9fad-4fb33afdbfad/458a1c59-d9de-4aa8-ac53-f47317918c09"
-					(reference "R20")
+					(reference "R24")
 					(unit 1)
 				)
@@
 		(on_board yes)
 		(dnp no)
-		(property "Reference" "#PWR086"
+		(property "Reference" "#PWR095"
 			(at 116.84 107.95 0)
 			(effects
@@
 			(project "EIM"
 				(path "/2e0b3b3d-5537-41dc-9fad-4fb33afdbfad/458a1c59-d9de-4aa8-ac53-f47317918c09"
-					(reference "#PWR086")
+					(reference "#PWR095")
 					(unit 1)
 				)
@@
 		(on_board yes)
 		(dnp no)
-		(property "Reference" "#PWR091"
+		(property "Reference" "#PWR0100"
 			(at 184.15 95.25 0)
 			(effects
@@
 			(project ""
 				(path "/2e0b3b3d-5537-41dc-9fad-4fb33afdbfad/458a1c59-d9de-4aa8-ac53-f47317918c09"
-					(reference "#PWR091")
-					(unit 1)
-				)
+					(reference "#PWR0100")
+					(unit 1)
+				)

Commit message: All components placed and pins assigned.
Parts:
- IC2: value SN65HVD1780QDRQ1 -> ISL3172EIBZ
- renumbered C43 to C35, D14 to D12, R22 to R17, R23 to R18, R24 to R19, R25 to R20, R26 to R21
Other:
- note added: "SN65HVD1780QDRQ1 is pin-to-pin replacement"
Changed lines of the file:
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@@
+		)
+	)
+	(text "SN65HVD1780QDRQ1 \nis pin-to-pin replacement"
+		(exclude_from_sim no)
+		(at 146.05 107.696 0)
+		(effects
+			(font
+				(size 1.27 1.27)
+			)
 		)
 	)
@@
 		(on_board yes)
 		(dnp no)
-		(property "Reference" "#PWR097"
+		(property "Reference" "#PWR090"
 			(at 166.37 74.93 0)
 			(effects
@@
 			(project "EIM"
 				(path "/2e0b3b3d-5537-41dc-9fad-4fb33afdbfad/458a1c59-d9de-4aa8-ac53-f47317918c09"
-					(reference "#PWR097")
+					(reference "#PWR090")
 					(unit 1)
 				)
@@
 			)
 		)
-		(property "Value" "SN65HVD1780QDRQ1"
+		(property "Value" "ISL3172EIBZ"
 			(at 146.05 86.36 0)
 			(effects
@@
 		(on_board yes)
 		(dnp no)
-		(property "Reference" "R23"
+		(property "Reference" "R18"
 			(at 125.984 67.056 0)
 			(effects
@@
 			(project "EIM"
 				(path "/2e0b3b3d-5537-41dc-9fad-4fb33afdbfad/458a1c59-d9de-4aa8-ac53-f47317918c09"
-					(reference "R23")
+					(reference "R18")
 					(unit 1)
 				)
@@
 		(on_board yes)
 		(dnp no)
-		(property "Reference" "R25"
+		(property "Reference" "R20"
 			(at 184.404 84.328 90)
 			(effects
@@
 			(project "EIM"
 				(path "/2e0b3b3d-5537-41dc-9fad-4fb33afdbfad/458a1c59-d9de-4aa8-ac53-f47317918c09"
-					(reference "R25")
+					(reference "R20")
 					(unit 1)
 				)
@@
 		(on_board yes)
 		(dnp no)
-		(property "Reference" "#PWR098"
+		(property "Reference" "#PWR091"
 			(at 166.37 88.9 0)
 			(effects
@@
 			(project "EIM"
 				(path "/2e0b3b3d-5537-41dc-9fad-4fb33afdbfad/458a1c59-d9de-4aa8-ac53-f47317918c09"
-					(reference "#PWR098")
+					(reference "#PWR091")
 					(unit 1)
 				)
@@
 		(on_board yes)
 		(dnp no)
-		(property "Reference" "C43"
+		(property "Reference" "C35"
 			(at 166.878 81.534 0)
 			(effects
@@
 			(project "EIM"
 				(path "/2e0b3b3d-5537-41dc-9fad-4fb33afdbfad/458a1c59-d9de-4aa8-ac53-f47317918c09"
-					(reference "C43")
+					(reference "C35")
 					(unit 1)
 				)
@@
 		(on_board yes)
 		(dnp no)
-		(property "Reference" "R26"
+		(property "Reference" "R21"
 			(at 184.404 102.108 90)
 			(effects
@@
 			(project "EIM"
 				(path "/2e0b3b3d-5537-41dc-9fad-4fb33afdbfad/458a1c59-d9de-4aa8-ac53-f47317918c09"
-					(reference "R26")
+					(reference "R21")
 					(unit 1)
 				)
@@
 		(on_board yes)
 		(dnp no)
-		(property "Reference" "#PWR096"
+		(property "Reference" "#PWR089"
 			(at 123.19 64.77 0)
 			(effects
@@
 			(project "EIM"
 				(path "/2e0b3b3d-5537-41dc-9fad-4fb33afdbfad/458a1c59-d9de-4aa8-ac53-f47317918c09"
-					(reference "#PWR096")
+					(reference "#PWR089")
 					(unit 1)
 				)
@@
 		(on_board yes)
 		(dnp no)
-		(property "Reference" "#PWR099"
+		(property "Reference" "#PWR092"
 			(at 166.37 111.76 0)
 			(effects
@@
 			(project "EIM"
 				(path "/2e0b3b3d-5537-41dc-9fad-4fb33afdbfad/458a1c59-d9de-4aa8-ac53-f47317918c09"
-					(reference "#PWR099")
+					(reference "#PWR092")
 					(unit 1)
 				)
@@
 		(dnp no)
 		(fields_autoplaced yes)
-		(property "Reference" "D14"
+		(property "Reference" "D12"
 			(at 196.85 93.9799 90)
 			(effects
@@
 			(project ""
 				(path "/2e0b3b3d-5537-41dc-9fad-4fb33afdbfad/458a1c59-d9de-4aa8-ac53-f47317918c09"
-					(reference "D14")
+					(reference "D12")
 					(unit 1)
 				)
@@
 		(on_board yes)
 		(dnp no)
-		(property "Reference" "R22"
+		(property "Reference" "R17"
 			(at 114.808 97.536 90)
 			(effects
@@
 			(project "EIM"
 				(path "/2e0b3b3d-5537-41dc-9fad-4fb33afdbfad/458a1c59-d9de-4aa8-ac53-f47317918c09"
-					(reference "R22")
+					(reference "R17")
 					(unit 1)
 				)
@@
 		(on_board yes)
 		(dnp no)
-		(property "Reference" "R24"
+		(property "Reference" "R19"
 			(at 160.02 126.238 90)
 			(effects
@@
 			(project "EIM"
 				(path "/2e0b3b3d-5537-41dc-9fad-4fb33afdbfad/458a1c59-d9de-4aa8-ac53-f47317918c09"
-					(reference "R24")
+					(reference "R19")
 					(unit 1)
 				)
@@
 		(on_board yes)
 		(dnp no)
-		(property "Reference" "#PWR095"
+		(property "Reference" "#PWR088"
 			(at 116.84 107.95 0)
 			(effects
@@
 			(project "EIM"
 				(path "/2e0b3b3d-5537-41dc-9fad-4fb33afdbfad/458a1c59-d9de-4aa8-ac53-f47317918c09"
-					(reference "#PWR095")
+					(reference "#PWR088")
 					(unit 1)
 				)
@@
 		(on_board yes)
 		(dnp no)
-		(property "Reference" "#PWR0100"
+		(property "Reference" "#PWR093"
 			(at 184.15 95.25 0)
 			(effects
@@
 			(project ""
 				(path "/2e0b3b3d-5537-41dc-9fad-4fb33afdbfad/458a1c59-d9de-4aa8-ac53-f47317918c09"
-					(reference "#PWR0100")
-					(unit 1)
-				)
+					(reference "#PWR093")
+					(unit 1)
+				)
