File: EIM/pcb/EIM/lowside_relay_driver.kicad_sch (KiCad schematic)
At the start: 1 part

Commit message: Layout 75% done, before 8V bus deletion
Changed lines of the file:
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@@
 	(text "input voltage above 2.3 V turns on\n"
 		(exclude_from_sim no)
-		(at 143.002 108.204 0)
+		(at 142.748 106.934 0)
 		(effects
 			(font
@@
 		(dnp no)
 		(fields_autoplaced yes)
-		(property "Reference" "#PWR0100"
+		(property "Reference" "#PWR0109"
 			(at 111.76 106.68 0)
 			(effects
@@
 			(project "EIM"
 				(path "/2e0b3b3d-5537-41dc-9fad-4fb33afdbfad/5bef9493-f8bd-441d-a08f-5b3ba2a87b31"
-					(reference "#PWR0100")
+					(reference "#PWR0109")
 					(unit 1)
 				)
 				(path "/2e0b3b3d-5537-41dc-9fad-4fb33afdbfad/e48675bc-9886-4777-98dd-45e1fd57f393"
-					(reference "#PWR0114")
+					(reference "#PWR0123")
 					(unit 1)
 				)
 				(path "/2e0b3b3d-5537-41dc-9fad-4fb33afdbfad/ff312e26-1222-4378-8a79-f4e4d02aafd2"
-					(reference "#PWR096")
+					(reference "#PWR0105")
 					(unit 1)
 				)
@@
 		(dnp no)
 		(fields_autoplaced yes)
-		(property "Reference" "#PWR0101"
+		(property "Reference" "#PWR0110"
 			(at 167.64 106.68 0)
 			(effects
@@
 			(project "EIM"
 				(path "/2e0b3b3d-5537-41dc-9fad-4fb33afdbfad/5bef9493-f8bd-441d-a08f-5b3ba2a87b31"
-					(reference "#PWR0101")
+					(reference "#PWR0110")
 					(unit 1)
 				)
 				(path "/2e0b3b3d-5537-41dc-9fad-4fb33afdbfad/e48675bc-9886-4777-98dd-45e1fd57f393"
-					(reference "#PWR0115")
+					(reference "#PWR0124")
 					(unit 1)
 				)
 				(path "/2e0b3b3d-5537-41dc-9fad-4fb33afdbfad/ff312e26-1222-4378-8a79-f4e4d02aafd2"
-					(reference "#PWR097")
+					(reference "#PWR0106")
 					(unit 1)
 				)
