File: VCU/temp_pcb/temp_vcu/CAN_transceiver.kicad_sch (KiCad schematic)
At the start: 5 parts, among them U3 SN65HVD233

Commit message: Ordered version of board
Parts:
- JP2: footprint Jumper:SolderJumper-2_P1.3mm_Open_RoundedPad1.0x1.5mm -> Connector_PinHeader_2.54mm:PinHeader_1x02_P2.54mm_Vertical
Changed lines of the file:
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@@
 			)
 		)
-		(property "Footprint" "Jumper:SolderJumper-2_P1.3mm_Open_RoundedPad1.0x1.5mm"
+		(property "Footprint" "Connector_PinHeader_2.54mm:PinHeader_1x02_P2.54mm_Vertical"
 			(at 143.51 120.65 0)
 			(effects
